File: neotron-1000.sch (KiCad schematic (older format))
At the start: 20 parts

Commit message: starting to change core and GPU
Parts:
- removed U?: STM32H743ZITx, Package_QFP:LQFP-144_20x20mm_P0.5mm, symbol MCU_ST_STM32H7:STM32H743ZITx
- removed U?: AS4C4M16SA, TSOPII-54, symbol Memory_RAM:AS4C4M16SA
- added J? (x2): USB_A, symbol Connector:USB_A
- added J?: Mini-DIN-6, symbol Connector:Mini-DIN-6
- gave numbers to parts that had none: 18
Connections:
- net GND: now also J2.11 (SHIELD), J3.13 (SHIELD), J?.3, J?.4 (GND), J?.4 (GND), J?.5 (Shield), J?.5 (Shield)
- net PS2_KBD_CLK: now also J?.5
- net PS2_KBD_DAT: now also J?.1
- net PS2_MSE_CLK: now also J?.6
- net PS2_MSE_DAT: now also J?.2
- net USB1_PWR: now also J?.1 (VBUS)
- net USB2_PWR: now also J?.1 (VBUS)
- net at U3.11 (DM1): now also J?.2 (D-)
- net at U3.12 (DP1): now also J?.3 (D+)
- net at U3.15 (DM2): now also J?.2 (D-)
- net at U3.16 (DP2): now also J?.3 (D+)
- new net +5V: J?.4
Other:
- note added: "Ethernet Controller & Port"
- note added: "PS2 Port"
- note added: "USB Hub & Ports"
- moved on the sheet: C1, C2, C3, FB1, J1, J2, J3, R1, R2, R3, R4, R5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
